File: VinoTemp/VinoTemp.brd (EAGLE design)
At the start: 124.5 x 20.3 mm, 32 parts, among them IC4 ATMEGA328, Y1 16MHz

Commit message: Fixed upside down LCD display
Parts:
- moved DOWN 40.0 mm to (69.2, 10.2)
- moved UP 40.0 mm to (109.2, 10.2)
- moved R10 19.3 mm to (97.8, 14.0), turned to 270 degrees
- moved R13 19.3 mm to (80.0, 6.35), turned to 270 degrees
- moved R17 19.3 mm to (80.0, 14.0), turned to 90 degrees
- moved R6 19.3 mm to (97.8, 6.35), turned to 90 degrees
- moved R11 14.8 mm to (82.5, 14.0), turned to 90 degrees
- moved R15 14.8 mm to (82.5, 6.35), turned to 270 degrees
- moved R4 14.8 mm to (95.2, 14.0), turned to 270 degrees
- moved R8 14.8 mm to (95.2, 6.35), turned to 90 degrees
- moved R14 10.8 mm to (85.1, 6.35), turned to 270 degrees
- moved R16 10.8 mm to (85.1, 14.0), turned to 90 degrees
- moved R7 10.8 mm to (92.7, 6.35), turned to 90 degrees
- moved R9 10.8 mm to (92.7, 14.0), turned to 270 degrees
- moved R12 8.03 mm to (87.6, 14.0), turned to 90 degrees
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Connections:
- net A2: now also DOWN.B2; no longer UP.B2
- net A3: now also UP.B2; no longer DOWN.B2
Routing:
- net VCC: track 162.5 -> 205.4 mm
- net D2: track 57.2 -> 94.0 mm
- net A1: track 76.7 -> 46.4 mm, vias 2 -> 1
- net D4: track 43.8 -> 73.7 mm, vias 1 -> 2
- net D7: track 31.9 -> 59.2 mm
- net D8: track 22.8 -> 47.9 mm
- net D12: track 71.1 -> 49.9 mm
- net D6: track 30.4 -> 49.5 mm
- net D10: track 53.8 -> 35.6 mm
- net D11: track 47.8 -> 31.1 mm, vias 1 -> 0
- net D5: track 35.5 -> 49.1 mm, vias 2 -> 1
- net D9: track 41.2 -> 27.9 mm
- net D13: track 51.8 -> 39.3 mm, vias 1 -> 0
- net A0: track 60.5 -> 49.0 mm
- net D3: track 60.2 -> 55.8 mm, vias 1 -> 3
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Other:
- board text added: "VinoTemp v2 - Aug 2015"
- board text removed: "VinoTemp v1 - Jul 2015"
