File: VinoTemp/VinoTemp.sch (EAGLE design)
At the start: 32 parts, among them IC4 ATMEGA328, Y1 16MHz

Commit message: Fixed upside down LCD display
Connections:
- net A2: now also DOWN.2; no longer UP.2
- net A3: now also UP.2; no longer DOWN.2
Other:
- moved on the sheet: DOWN, UP
